File: mPCIe-GNSS.sch (KiCad schematic (older format))
At the start: 23 parts, among them J1 1PPS, J2 ANT, Q1 DTC143Z, Q2 DTA043T, U1 FT234XD-T

Commit message: version 0.3
Parts:
- removed U1: FT234XD-T, L80:SON45P300X300X80-13N, symbol CustomDevice:FT234XD-T
- added C7: 4.7uF, Capacitor_SMD:C_0402_1005Metric, symbol Device:C
- added C8: 100nF, Capacitor_SMD:C_0402_1005Metric, symbol Device:C
- added C9: 1uF, Capacitor_SMD:C_0402_1005Metric, symbol Device:C
- added R7: 4.7K, Resistor_SMD:R_0402_1005Metric, symbol Device:R
- added U1: CP2102N-A01-GQFN28, QFN28G_0.5-5X5MM, symbol INTERFACE-CP2102-GMR_QFN28_:CP2102-GMR(QFN28)
- C1: value XH414HG -> DSK-3R3H224U-HL; footprint L80:CAP_XH414H-IV01E -> 1 My Footprints:CAP_DSK-3R3H224U-HL
- C2: footprint Capacitor_SMD:C_0603_1608Metric_Pad1.05x0.95mm_HandSolder -> Capacitor_SMD:C_0402_1005Metric; LCSC (none) -> C23733
- C3: footprint Capacitor_SMD:C_0603_1608Metric_Pad1.05x0.95mm_HandSolder -> Capacitor_SMD:C_0402_1005Metric; LCSC (none) -> C1525
- C4: renamed from C6; footprint Capacitor_SMD:C_0603_1608Metric_Pad1.05x0.95mm_HandSolder -> Capacitor_SMD:C_0402_1005Metric; LCSC (none) -> C1525
- C5: footprint Capacitor_SMD:C_0603_1608Metric_Pad1.05x0.95mm_HandSolder -> Capacitor_SMD:C_0402_1005Metric; LCSC (none) -> C15525
- C6: renamed from C4; footprint Capacitor_SMD:C_0603_1608Metric_Pad1.05x0.95mm_HandSolder -> Capacitor_SMD:C_0402_1005Metric; LCSC (none) -> C1525
- D1: LCSC (none) -> C154821
- GNSS1: footprint L80:XCVR_LC86L -> 1 My Footprints:XCVR_LC86L
- J1: footprint Connector_JST:JST_SHL_SM02B-SHLS-TF_1x02-1MP_P1.00mm_Horizontal -> 1 My Footprints:JST_SH_SM02B-SRSS-TB_1x02-1MP_P1.00mm_Horizontal_3D
- LED1: footprint LED_SMD:LED_0603_1608Metric_Pad1.05x0.95mm_HandSolder -> 1 My Footprints:LED_0603_1608Metric_SnapModel; LCSC (none) -> C72041
- LED2: footprint LED_SMD:LED_0603_1608Metric_Pad1.05x0.95mm_HandSolder -> 1 My Footprints:LED_0603_1608Metric_SnapModel; LCSC (none) -> C72038
- LED3: footprint LED_SMD:LED_0603_1608Metric_Pad1.05x0.95mm_HandSolder -> 1 My Footprints:LED_0603_1608Metric_SnapModel; LCSC (none) -> C72043
- PC1: footprint mini-PCIe Cards:mini-PCIe_F1_Full -> mini-PCIe Cards:mini-PCIe_F1_Full_v517
- Q1: footprint Package_TO_SOT_SMD:SC-59_Handsoldering -> 1 My Footprints:Q_EMT3F
- Q2: footprint L80:Q-EMT3 -> 1 My Footprints:Q_EMT3F
- R1: footprint Resistor_SMD:R_0603_1608Metric_Pad1.05x0.95mm_HandSolder -> Resistor_SMD:R_0402_1005Metric; LCSC (none) -> C11702
- R2, R3: value 27R -> 33R; footprint Resistor_SMD:R_0603_1608Metric_Pad1.05x0.95mm_HandSolder -> Resistor_SMD:R_0402_1005Metric; LCSC (none) -> C25105
- R4: value 1K -> 51R; footprint Resistor_SMD:R_0603_1608Metric_Pad1.05x0.95mm_HandSolder -> Resistor_SMD:R_0402_1005Metric; LCSC (none) -> C25125
- R5, R6: value 1K -> 220R; footprint Resistor_SMD:R_0603_1608Metric_Pad1.05x0.95mm_HandSolder -> Resistor_SMD:R_0402_1005Metric; LCSC (none) -> C25091
Connections:
- net FT_D+ is gone; now on net USB_D+: R2.1
- net FT_D- is gone; now on net USB_D-: R3.2
- net +3V3: now also C6.2, C7.1, C8.2, C9.1, R7.1, U1.6 (VDD), U1.7 (REGIN), U1.8 (VBUS); no longer C6.1
- net 1PPS: now also U1.23 (CTS)
- net GND: now also C6.1, PC1.54 (MOUNT1), PC1.55 (MOUNT2), C7.2, C8.1, C9.2, U1.29 (GND), U1.3 (GND); no longer C6.2
- net GPS_RX: now also U1.26 (TXD)
- net GPS_TX: now also U1.25 (RXD)
- net USB_D+: no longer R2.2
- net USB_D-: no longer R3.1
- net +BATT renamed VBAT
- net LED_WLAN renamed ~LED_WLAN
- net RESET renamed ~RESET
- net ~RESET: now also R7.2, U1.9 (~RST)
- new net U232_D+: R2.2, U1.4 (D+)
- new net U232_D-: R3.1, U1.5 (D-)
- no-connect marks 27 -> 31
Other:
- moved on the sheet: C1, C2, C3, C4, C5, C6, D1, GNSS1, J1, J2, LED1, LED2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
