File: mPCIe-GNSS/mPCIe-GNSS.sch (KiCad schematic (older format))
At the start: 27 parts, among them J1 1PPS, J2 ANT, Q1 DTC143Z, Q2 DTA043T, U1 CP2102N-A01-GQFN28

Commit message: restructure
Parts:
- GNSS1: symbol L80:LC86L -> mPCIe-GNSS-rescue:LC86L-L80
- PC1: symbol mPCIe:miniPCIe -> mPCIe-GNSS-rescue:miniPCIe-mPCIe
- U1: symbol INTERFACE-CP2102-GMR_QFN28_:CP2102-GMR(QFN28) -> mPCIe-GNSS-rescue:CP2102-GMR(QFN28)-INTERFACE-CP2102-GMR_QFN28_
Changed lines of the file:
@@
 $EndDescr
 $Comp
-L mPCIe:miniPCIe PC1
+L mPCIe-GNSS-rescue:miniPCIe-mPCIe PC1
 U 1 1 5FF82652
 P 2000 4200
@@
 $EndComp
 $Comp
-L L80:LC86L GNSS1
+L mPCIe-GNSS-rescue:LC86L-L80 GNSS1
 U 1 1 5FF86FE8
 P 5450 2250
@@
 GND
 $Comp
-L INTERFACE-CP2102-GMR_QFN28_:CP2102-GMR(QFN28) U1
+L mPCIe-GNSS-rescue:CP2102-GMR(QFN28)-INTERFACE-CP2102-GMR_QFN28_ U1
 U 1 1 600D508D
 P 5950 4500
